File: HW/SAR-APRS/SAR-APRS.kicad_pcb (KiCad board)
At the start: 2 copper layers, 5 parts, among them J1 uFl, Q1 2N7002, U1 DRA818V, U2 arduino_mini_clone, U4 HC-05

Commit message: update
Parts:
- added J4: uFl, w_conn_rf:coaxial_u.fl-r-smt-1, F.Cu at (188.6, 58.7)
Changed lines of the file:
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@@
     (tracks 0)
     (zones 0)
-    (modules 5)
-    (nets 50)
+    (modules 6)
+    (nets 51)
   )
   (page A4)
@@
   (net 48 "Net-(R11-Pad2)")
   (net 49 "Net-(R12-Pad1)")
+  (net 50 "Net-(J4-Pad1)")
   (net_class Default "This is the default net class."
     (clearance 0.2)
@@
     (add_net "Net-(J2-Pad3)")
     (add_net "Net-(J2-Pad4)")
+    (add_net "Net-(J4-Pad1)")
     (add_net "Net-(Q1-Pad1)")
     (add_net "Net-(Q1-Pad3)")
@@
     (add_net "Net-(U4-Pad11)")
   )
+  (module w_conn_rf:coaxial_u.fl-r-smt-1 (layer F.Cu)
+    (at 188.6 58.7)
+    (descr "Ultra small surface mount coaxial connector, Hirose U.FL-R-SMT-1")
+    (fp_text reference J4 (at 0 -2.1) (layer F.SilkS)
+      (effects (font (size 0.5 0.5) (thickness 0.1)))
+    )
+    (fp_text value uFl (at 0 2.7) (layer F.SilkS)
+      (effects (font (size 0.5 0.5) (thickness 0.1)))
+    )
+    (fp_arc (start -1 -1) (end -1.3 -1) (angle 90) (layer F.SilkS) (width 0.15))
+    (fp_arc (start 1 -1) (end 1 -1.3) (angle 90) (layer F.SilkS) (width 0.15))
+    (fp_arc (start 1 1) (end 1.3 1) (angle 90) (layer F.SilkS) (width 0.15))
+    (fp_arc (start -1 1) (end -1 1.3) (angle 90) (layer F.SilkS) (width 0.15))
+    (fp_line (start -1 -1.3) (end 1 -1.3) (layer F.SilkS) (width 0.15))
+    (fp_line (start 1.3 -1) (end 1.3 1) (layer F.SilkS) (width 0.15))
+    (fp_line (start 1 1.3) (end -1 1.3) (layer F.SilkS) (width 0.15))
+    (fp_line (start -1.3 1) (end -1.3 -1) (layer F.SilkS) (width 0.15))
+    (fp_circle (center 0 0) (end -1 0) (layer F.SilkS) (width 0.15))
+    (fp_circle (center 0 0) (end -0.1 0) (layer F.SilkS) (width 0.15))
+    (pad 1 smd rect (at 0 1.525) (size 1 1.05) (layers F.Cu F.Paste F.Mask)
+      (net 50 "Net-(J4-Pad1)") (solder_mask_margin 0.07) (solder_paste_margin -0.05))
+    (pad 2 smd rect (at 1.475 0) (size 1.05 2.2) (layers F.Cu F.Paste F.Mask)
+      (net 44 Bat-) (solder_mask_margin 0.07) (solder_paste_margin -0.05))
+    (pad 2 smd rect (at -1.475 0) (size 1.05 2.2) (layers F.Cu F.Paste F.Mask)
+      (net 44 Bat-) (solder_mask_margin 0.07) (solder_paste_margin -0.05))
+    (model walter/conn_rf/coaxial_u.fl-r-smt-1.wrl
+      (at (xyz 0 0 0))
+      (scale (xyz 1 1 1))
+      (rotate (xyz 0 0 0))
+    )
+  )
   (module "maxrez:HC-05 BT" (layer F.Cu)

Commit message: schematic update memmory adding
Parts:
- added U7: AT45DB641, Mlab_IO:SOIC-8_3.9x4.9mm_Pitch1.27mm, F.Cu at (184.3, 73.5)

Commit message: schem and pcb update
Parts:
- added C1: 100nF, Capacitors_SMD:C_0603, F.Cu at (198.0, 95.0)
- added C2: 10uF, Capacitors_SMD:C_0603, F.Cu at (198.0, 98.0)
- added C3: 20pF, Capacitors_SMD:C_0805, F.Cu at (241.5, 69.5)
- added C4: 36pF, Capacitors_SMD:C_0805, F.Cu at (237.5, 76.0)
- added C5: 36pF, Capacitors_SMD:C_0805, F.Cu at (237.5, 82.5)
- added C6: 20pF, Capacitors_SMD:C_0805, F.Cu at (241.5, 89.0)
- added C7: 100nF, Capacitors_SMD:C_0603, F.Cu at (211.0, 66.0)
- added L1: 56nH, Inductors_SMD:L_0805, F.Cu at (239.5, 73.0)
- added L2: 68nH, Inductors_SMD:L_0805, F.Cu at (238.5, 79.5)
- added L3: 56nH, Inductors_SMD:L_0805, F.Cu at (239.5, 85.5)
- added Q2: 2N7002, TO_SOT_Packages_SMD:SOT-23, F.Cu at (167.1, 76.6)
- added Q3: 2N7002, TO_SOT_Packages_SMD:SOT-23, F.Cu at (167.1, 81.2)
- added R1: 620, Resistors_SMD:R_0603, F.Cu at (200.5, 97.5)
- added R2: 4k7, Resistors_SMD:R_0603, F.Cu at (225.0, 66.5)
- added R3: 100k, Resistors_SMD:R_0603, F.Cu at (213.0, 63.5)
- added R4: 100k, Resistors_SMD:R_0603, F.Cu at (209.0, 63.5)
- added R5: 10k, Resistors_SMD:R_0603, F.Cu at (220.0, 62.0)
- added RV1: 100k, Potentiometers:Potentiometer_Trimmer-EVM3E, F.Cu at (202.0, 93.5)
- added U3: DW01x, Mlab_IO:SOT-23-6, F.Cu at (161.7, 30.9)
- added U5: AT45DB641, Mlab_IO:SOIC-8_3.9x4.9mm_Pitch1.27mm, F.Cu at (120.0, 84.6)
- added U6: ATMEGA328-AU, Housings_QFP:TQFP-32_7x7mm_Pitch0.8mm, F.Cu at (182.5, 79.0)
- added U8: HC-05, maxrez:HC-05 BT, F.Cu at (102.1, 54.1)
- U2: value arduino_mini_clone -> TP4056; footprint APRS_modules:arduino_mini_clone -> IO:SO-8_3.9x4.9mm_P1.27mm
- U4: value HC-05 -> ADP1108AN-3.3; footprint maxrez:HC-05 BT -> Housings_SOIC:SOIC-8_3.9x4.9mm_Pitch1.27mm
- U7: value AT45DB641 -> CH340C; footprint Mlab_IO:SOIC-8_3.9x4.9mm_Pitch1.27mm -> IO:SOP-16_4.55x10.3mm_P1.27mm
- moved J1 69.4 mm to (238.5, 64.5)
- moved U2 64.3 mm to (155.6, 31.9)
- moved J4 62.9 mm to (130.7, 83.2)
- moved Q1 47.2 mm to (220.0, 65.0), turned to 270 degrees
- moved U1 30.5 mm to (215.5, 79.0)
- moved U4 23.1 mm to (155.6, 76.4)
- moved U7 14.6 mm to (186.3, 59.0)
Connections:
- J1 pad 2: Bat- -> GND
- J4 pad 2: Bat- -> GND
- Q1 pad 1: Net-(Q1-Pad1) -> /CPU/RFMOD_PTT
- Q1 pad 2: Bat- -> GND
- U1 pad 10: Bat- -> GND
- U1 pad 16: Net-(U1-Pad16) -> /RF_MODULE/RFMOD_RXD
- U1 pad 17: Net-(U1-Pad17) -> /CPU/RFMOD_RXD
- U1 pad 8: Bat+ -> +3V3
- U1 pad 9: Bat- -> GND
- U1 pad P2: Bat- -> GND
- U1 pad P3: Bat- -> GND
- U2 pad 1: Bat- -> GND
- U2 pad 3: Net-(U2-Pad3) -> GND
- U2 pad 4: Net-(U2-Pad4) -> Net-(C9-Pad1)
- U2 pad 5: Net-(U2-Pad5) -> Bat+
- U2 pad 6: Net-(U1-Pad16) -> Net-(R8-Pad1)
- U2 pad 7: Net-(U1-Pad17) -> Net-(R9-Pad1)
- U2 pad 8: Net-(C7-Pad1) -> Net-(C9-Pad1)
- U4 pad 1: Net-(U2-Pad29) -> Net-(R12-Pad1)
- U4 pad 2: Net-(U2-Pad28) -> Bat+
- U4 pad 3: (no net) -> Net-(D2-Pad2)
- U4 pad 4: (no net) -> GND
- U4 pad 5: (no net) -> GND
- U4 pad 6: (no net) -> Net-(U4-Pad6)
- U4 pad 7: (no net) -> Net-(U4-Pad7)
- U4 pad 8: (no net) -> Net-(R13-Pad1)
- U7 pad 1: Net-(U2-Pad4) -> GND
- U7 pad 2: Net-(U2-Pad33) -> /CPU/TXD
- U7 pad 3: +3V3 -> /CPU/RXD
- U7 pad 4: Bat- -> +3V3
- U7 pad 6: +3V3 -> Net-(J2-Pad2)
- U7 pad 7: Bat- -> Net-(U7-Pad7)
- U7 pad 8: Net-(U2-Pad5) -> Net-(U7-Pad8)
