File: HW/SAR-APRS/SAR-APRS.kicad_pcb (KiCad board)
At the start: 2 copper layers, 29 parts, among them J1 uFl, J4 uFl, Q1 2N7002, Q2 2N7002, Q3 2N7002, U1 DRA818V, U2 TP4056, U3 DW01x, U4 ADP1108AN-3.3, U5 AT45DB641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

Commit message: schm and pcb update
Parts:
- added C10: 100nF, Capacitors_SMD:C_0603, F.Cu at (178.2, -10.1)
- added C13: 100nF, Capacitors_SMD:C_0603, F.Cu at (169.9, -13.0)
- added C14: 100nF, Capacitors_SMD:C_0603, F.Cu at (211.2, 102.4)
- added C15: 100nF, Capacitors_SMD:C_0603, F.Cu at (211.2, 100.8)
- added C16: 100nF, Capacitors_SMD:C_0603, F.Cu at (218.8, 100.0)
- added C17: 22pF, Capacitors_SMD:C_0603, F.Cu at (162.2, -13.0)
- added C18: 100nF, Capacitors_SMD:C_0603, F.Cu at (218.8, 101.6)
- added C19: 100nF, Capacitors_SMD:C_0603, F.Cu at (162.2, -10.7)
- added C20: 22pF, Capacitors_SMD:C_0603, F.Cu at (166.1, -13.0)
- added C21: 100nF, Capacitors_SMD:C_0603, F.Cu at (158.4, -5.95)
- added C22: 100nF, Capacitors_SMD:C_0603, F.Cu at (158.4, -0.49)
- added C23: 100nF, Capacitors_SMD:C_0603, F.Cu at (178.2, -4.56)
- added C24: 100nF, Capacitors_SMD:C_0603, F.Cu at (178.2, -2.21)
- added C25: 100nF, Capacitors_SMD:C_0603, F.Cu at (182.1, -4.56)
- added C27: 100nF, Capacitors_SMD:C_0603, F.Cu at (166.1, -10.7)
- added C9: 100nF, Capacitors_SMD:C_0603, F.Cu at (184.0, -13.0)
- added D1: LED, LEDs:LED_0603, F.Cu at (122.0, -2.00)
- added D2: LED, LEDs:LED_0603, F.Cu at (122.0, 0.35)
- added D4: LED, LEDs:LED_0603, F.Cu at (133.4, -2.00)
- added J2: USB_B_Mini, Connectors:USB_Mini-B, F.Cu at (200.7, 139.3)
- added L5: L_Small, Inductors_SMD:L_0805, F.Cu at (235.0, -4.00)
- added R10: 100, Resistors_SMD:R_0603, F.Cu at (185.0, -37.0)
- added R11: 1k, Resistors_SMD:R_0603, F.Cu at (188.6, -37.0)
- added R15: 1k, Resistors_SMD:R_0603, F.Cu at (222.1, -4.29)
- added R16: 10k, Resistors_SMD:R_0603, F.Cu at (222.1, -1.80)
- added R17: 3k3, Resistors_SMD:R_0603, F.Cu at (225.6, -4.29)
- added R20: 1k, Resistors_SMD:R_0603, F.Cu at (225.6, -1.80)
- added R23: 100k, Resistors_SMD:R_0603, F.Cu at (222.1, 4.11)
- added R24: 100k, Resistors_SMD:R_0603, F.Cu at (222.1, 6.58)
- added R25: 100k, Resistors_SMD:R_0603, F.Cu at (225.6, 4.11)
- added R26: 100, Resistors_SMD:R_0603, F.Cu at (238.9, -4.29)
- added R27: 1k, Resistors_SMD:R_0603, F.Cu at (238.9, -1.80)
- added R6: 0.4, Resistors_SMD:R_2512, F.Cu at (179.2, -12.7)
- added R7: 1k2, Resistors_SMD:R_0603, F.Cu at (181.9, -10.1)
- added R8: 1k, Resistors_SMD:R_0603, F.Cu at (234.2, 4.11)
- added R9: 1k, Resistors_SMD:R_0603, F.Cu at (237.8, 4.11)
- added U9: NEO_GPS_MODULE, Mlab_Pin_Headers:Straight_1x04, F.Cu at (222.1, 138.7)
- moved U7 61.6 mm to (210.3, 115.7)
- moved U6 56.8 mm to (225.9, 115.6), turned to 0 degrees

Commit message: PCB update
Parts:
- added C11: 10uF, Capacitors_SMD:C_1210, F.Cu at (125.9, 139.6)
- added C12: 10uF, Capacitors_SMD:C_1210, F.Cu at (145.5, 130.7)
- added C26: 10uF, Capacitors_SMD:C_1210, F.Cu at (118.0, 80.8)
- added C8: 10uF, Capacitors_SMD:C_1210, F.Cu at (120.8, 129.3)
- added D3: MBRS130T3G, Diodes_SMD:D_SMB, F.Cu at (145.5, 137.3)
- added D6: LED, LEDs:LED_0805, F.Cu at (106.6, 120.5)
- added D7: LED, LEDs:LED_0805, F.Cu at (112.1, 59.4)
- added J3: JTAG, Mlab_Pin_Headers:Straight_2x03, F.Cu at (141.6, 120.0)
- added J5: OLED, Mlab_Pin_Headers:Straight_1x04, F.Cu at (142.9, 110.5)
- added J6: HEADER_1x02, Mlab_Pin_Headers:Straight_1x02, F.Cu at (118.8, 142.3)
- added L4: 22uH, Inductors_SMD:L_6.3x6.3_H3, F.Cu at (137.7, 145.0)
- added R12: ?, Resistors_SMD:R_0805, F.Cu at (135.3, 140.0)
- added R13: 2k4, Resistors_SMD:R_0805, F.Cu at (141.1, 132.1)
- added R14: 1k5, Resistors_SMD:R_0805, F.Cu at (141.1, 129.8)
- added R18: 2K, Resistors_SMD:R_0805, F.Cu at (137.1, 105.4)
- added R19: 330, Resistors_SMD:R_0805, F.Cu at (132.0, 103.0)
- added R21: 620, Resistors_SMD:R_0805, F.Cu at (118.0, 103.0)
- added SW1: SW_DPST_x2, Buttons_Switches_SMD:SW_SPST_EVQP0, F.Cu at (111.0, 101.0)
- added SW2: SW_DPST_x2, Buttons_Switches_SMD:SW_SPST_EVQP0, F.Cu at (125.0, 101.0)
- added SW3: SW_DPST_x2, Buttons_Switches_SMD:SW_SPST_EVQP0, F.Cu at (139.0, 101.0)
- added U10: NEO-M8, RF_GPS:ublox_NEO, F.Cu at (110.6, 69.4)
- added U11: EEPROM, IO:TSSOP-8_4.4x3mm_P0.65mm, F.Cu at (107.4, 80.0)
- added Y1: 16MHz, Mlab_XTAL:ISM81, F.Cu at (119.9, 120.0)
- C1, C10, C13, C14, C15, C16, C17, C18, C19, C2, C20, C21, C22, C23, C24, C25, C27, C7, C9: footprint Capacitors_SMD:C_0603 -> Capacitors_SMD:C_0805
- D1, D2, D4: footprint LEDs:LED_0603 -> LEDs:LED_0805
- J1: footprint w_conn_rf:coaxial_u.fl-r-smt-1 -> w_conn_rf:sma_straight_32k101-400l5
- R1, R10, R11, R15, R16, R17, R2, R20, R23, R24, R25, R26, R27, R3, R4, R5, R7, R8, R9: footprint Resistors_SMD:R_0603 -> Resistors_SMD:R_0805
- RV1: footprint Potentiometers:Potentiometer_Trimmer-EVM3E -> Potentiometers:Potentiometer_Trimmer_Bourns_3214J
- U1: value DRA818V -> U1
- U8: moved to B.Cu
- moved R11 188.6 mm to (129.3, 142.1), turned to 270 degrees
- moved R10 188.4 mm to (122.2, 140.6), turned to 90 degrees
- moved R9 168.1 mm to (130.2, 133.3)
- moved R8 167.6 mm to (130.2, 135.6)
- moved R25 164.8 mm to (106.8, 118.3)
- moved C10 164.1 mm to (122.2, 144.1), turned to 270 degrees
- moved C9 162.8 mm to (119.2, 136.3), turned to 90 degrees
- moved R6 160.0 mm to (116.1, 134.3), turned to 90 degrees
- moved R23 158.9 mm to (106.8, 113.5), turned to 180 degrees
- moved R24 158.9 mm to (106.8, 115.9), turned to 180 degrees
- moved R7 156.0 mm to (119.2, 132.8), turned to 90 degrees
- moved C27 154.9 mm to (103.6, 131.1), turned to 90 degrees
- moved R26 147.0 mm to (106.9, 60.5), turned to 270 degrees
- moved R17 145.8 mm to (136.6, 111.2)
- moved C19 145.8 mm to (114.9, 127.3), turned to 90 degrees
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Connections:
- R27 pad 2: /GPS/GPS_PPS -> /CPU/GPS_PPS
- U1 pad 16: /RF_MODULE/RFMOD_RXD -> /CPU/RFMOD_RXD
- U1 pad 17: /CPU/RFMOD_RXD -> /CPU/RFMOD_TXD
- U6 pad 1: /CPU/RFMOD_RXD -> /CPU/RFMOD_TXD
- U6 pad 10: /CPU/BT_TXD -> /BT_module/BT_TXD
- U6 pad 12: /CPU/BT_LED2 -> /BT_module/BT_LED2
- U6 pad 25: /CPU/OLED_SDA -> /CPU/OLED_SCL
- U6 pad 26: /CPU/OLED_SCL -> /CPU/OLED_SDA
- U6 pad 27: Net-(U6-Pad27) -> /CPU/BUTTON
- U6 pad 28: Net-(U6-Pad28) -> /CPU/LED
- U6 pad 32: /RF_MODULE/RFMOD_RXD -> /CPU/RFMOD_RXD
- U7 pad 2: /CPU/TXD -> /GPS/GPS_RXD
- U7 pad 3: /CPU/RXD -> /CPU/GPS_RXD
- U8 pad 1: /BT_module/BD_TXD -> /BT_module/BT_TXD
Routing:
- net +3V3: track 0.00 -> 257.6 mm, vias 0 -> 5
- net Bat+: track 0.00 -> 94.4 mm
- net /CPU/GPS_RXD: track 0.00 -> 75.2 mm, vias 0 -> 1
- net /GPS/GPS_RXD: track 0.00 -> 73.2 mm, vias 0 -> 1
- net /CPU/GPS_PPS: track 0.00 -> 65.0 mm, vias 0 -> 2
- net /CPU/RESET: track 0.00 -> 59.3 mm, vias 0 -> 2
- net /CPU/RFMOD_PTT: track 0.00 -> 57.3 mm, vias 0 -> 2
- net /CPU/RFMOD_AUX: track 0.00 -> 41.8 mm, vias 0 -> 2
- net /CPU/RFMOD_RXD: track 0.00 -> 40.3 mm, vias 0 -> 2
- net /CPU/RFMOD_TXD: track 0.00 -> 39.6 mm, vias 0 -> 2
- net /BT_module/BT_CMD: track 0.00 -> 32.0 mm, vias 0 -> 2
- net /CPU/VUSB: track 0.00 -> 28.0 mm, vias 0 -> 4
- net /BT_module/BT_LED2: track 0.00 -> 28.0 mm, vias 0 -> 2
- net Net-(C9-Pad1): track 0.00 -> 26.5 mm
- net GND: track 0.00 -> 24.5 mm, vias 0 -> 138
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- added copper zone on B.Cu, net GND
- added copper zone on F.Cu, net GND
Other:
- board outline added: 50 x 100 mm
- board text added: "+3V3"
- board text added: "GND"
- board text added: "J1"
- board text added: "J4"
- board text added: "J5"
- board text added: "MISO"
- board text added: "MOSI"
- board text added: "RST"
- board text added: "RV1"
- board text added: "RXD"
- board text added: "SAR_APRS V 1.0"
- board text added: "SCK"
- board text added: "SCL"
- board text added: "SDA"
- board text added: "TXD"
- board text added: "U3"
- board text added: "U5"
- board text added: "U8"
- board text added: "Y1"
