File: HW/SAR-APRS/Power.sch (KiCad schematic (older format))
At the start: 23 parts, among them Q2 2N7002, Q3 2N7002, U2 TP4056, U3 DW01x, U4 ADP1108AN-3.3

Commit message: PCB update
Parts:
- removed C11: 10uF, symbol device:C_Small
- added C11: 10uF, Capacitors_SMD:C_1210, symbol device:CP1_Small
- added J6: HEADER_1x02, Mlab_Pin_Headers:Straight_1x02, symbol MLAB_HEADER:HEADER_1x02
- C10, C9: footprint Capacitors_SMD:C_0603 -> Capacitors_SMD:C_0805
- C12, C8: footprint (none) -> Capacitors_SMD:C_1210
- D1, D2: footprint LEDs:LED_0603 -> LEDs:LED_0805
- D3: value 1N5818 -> MBRS130T3G; footprint Diode_THT:D_DO-41_SOD81_P10.16mm_Horizontal -> Diodes_SMD:D_SMB
- L4: footprint (none) -> Inductors_SMD:L_6.3x6.3_H3
- R10, R11, R7, R8, R9: footprint Resistors_SMD:R_0603 -> Resistors_SMD:R_0805
- R12, R13, R14: footprint (none) -> Resistors_SMD:R_0805
Connections:
- net Bat+: now also C11.1, J6.1
- net Bat-: now also J6.2
- net GND: now also C11.2
Other:
- note added: "footprint ok"
- moved on the sheet: L4
Changed lines of the file:
@@
 F 0 "R7" V 6475 1800 50  0000 L CNN
 F 1 "1k2" V 6475 1975 50  0000 L CNN
-F 2 "Resistors_SMD:R_0603" H 6575 1975 50  0001 C CNN
+F 2 "Resistors_SMD:R_0805" H 6575 1975 50  0001 C CNN
 F 3 "~" H 6575 1975 50  0001 C CNN
 	1    6575 1975
 	0    -1   1    0
-$EndComp
-$Comp
-L device:C_Small C?
-U 1 1 5C95AC48
-P 6825 3550
-AR Path="/5C95AC48" Ref="C?"  Part="1"
-AR Path="/5C948828/5C95AC48" Ref="C11"  Part="1"
-F 0 "C11" H 6925 3575 50  0000 L CNN
-F 1 "10uF" H 6875 3475 50  0000 L CNN
-F 2 "" H 6825 3550 50  0001 C CNN
-F 3 "~" H 6825 3550 50  0001 C CNN
-	1    6825 3550
-	1    0    0    -1
 $EndComp
 $Comp
@@
 Wire Wire Line
 	5000 1875 5050 1875
-Text GLabel 6950 3250 2    50   Input ~ 0
+Text GLabel 7475 3250 2    50   Input ~ 0
 Bat+
-Text GLabel 6950 4050 2    50   Input ~ 0
+Text GLabel 7475 4050 2    50   Input ~ 0
 Bat-
 Wire Wire Line
@@
 F 0 "R9" H 4850 2950 50  0000 L CNN
 F 1 "1k" H 4900 3025 50  0000 L CNN
-F 2 "Resistors_SMD:R_0603" H 5050 2975 50  0001 C CNN
+F 2 "Resistors_SMD:R_0805" H 5050 2975 50  0001 C CNN
 F 3 "~" H 5050 2975 50  0001 C CNN
 	1    5050 2975
@@
 F 0 "R8" H 4900 2950 50  0000 L CNN
 F 1 "1k" H 4950 3025 50  0000 L CNN
-F 2 "Resistors_SMD:R_0603" H 4850 2975 50  0001 C CNN
+F 2 "Resistors_SMD:R_0805" H 4850 2975 50  0001 C CNN
 F 3 "~" H 4850 2975 50  0001 C CNN
 	1    4850 2975
@@
 F 0 "C10" H 6575 3325 50  0000 L CNN
 F 1 "100nF" H 6550 3225 50  0000 L CNN
-F 2 "Capacitors_SMD:C_0603" H 6475 3350 50  0001 C CNN
+F 2 "Capacitors_SMD:C_0805" H 6475 3350 50  0001 C CNN
 F 3 "~" H 6475 3350 50  0001 C CNN
 	1    6475 3350
@@
 F 0 "R10" H 6734 3296 50  0000 L CNN
 F 1 "100" H 6725 3200 50  0000 L CNN
-F 2 "Resistors_SMD:R_0603" H 6675 3250 50  0001 C CNN
+F 2 "Resistors_SMD:R_0805" H 6675 3250 50  0001 C CNN
 F 3 "~" H 6675 3250 50  0001 C CNN
 	1    6675 3250
@@
 F 0 "R11" H 5559 3796 50  0000 L CNN
 F 1 "1k" H 5550 3700 50  0000 L CNN
-F 2 "Resistors_SMD:R_0603" H 5500 3750 50  0001 C CNN
+F 2 "Resistors_SMD:R_0805" H 5500 3750 50  0001 C CNN
 F 3 "~" H 5500 3750 50  0001 C CNN
 	1    5500 3750
@@
 F 0 "C9" H 6575 2475 50  0000 L CNN
 F 1 "100nF" H 6550 2375 50  0000 L CNN
-F 2 "Capacitors_SMD:C_0603" H 6475 2500 50  0001 C CNN
+F 2 "Capacitors_SMD:C_0805" H 6475 2500 50  0001 C CNN
 F 3 "~" H 6475 2500 50  0001 C CNN
 	1    6475 2500
@@
 	6825 3250 6775 3250
 Wire Wire Line
-	6950 3250 6825 3250
+	7475 3250 7325 3250
 Connection ~ 6825 3250
 Wire Wire Line
-	6475 4050 6950 4050
+	6475 4050 7325 4050
 Connection ~ 6475 4050
 $Comp
@@
 AR Path="/5C948828/5C95ACFC" Ref="D3"  Part="1"
 F 0 "D3" H 6150 4734 50  0000 C CNN
-F 1 "1N5818" H 6150 4825 50  0000 C CNN
-F 2 "Diode_THT:D_DO-41_SOD81_P10.16mm_Horizontal" H 6150 4775 50  0001 C CNN
+F 1 "MBRS130T3G" H 6150 4825 50  0000 C CNN
+F 2 "Diodes_SMD:D_SMB" H 6150 4775 50  0001 C CNN
 F 3 "http://www.vishay.com/docs/88525/1n5817.pdf" H 6150 4950 50  0001 C CNN
 	1    6150 4950
@@
 L device:L_Small L?
 U 1 1 5C95AD02
-P 5775 4950
+P 5700 4950
 AR Path="/5C95AD02" Ref="L?"  Part="1"
 AR Path="/5C948828/5C95AD02" Ref="L4"  Part="1"
-F 0 "L4" V 5960 4950 50  0000 C CNN
-F 1 "22uH" V 5869 4950 50  0000 C CNN
-F 2 "" H 5775 4950 50  0001 C CNN
-F 3 "~" H 5775 4950 50  0001 C CNN
-	1    5775 4950
+F 0 "L4" V 5885 4950 50  0000 C CNN
+F 1 "22uH" V 5794 4950 50  0000 C CNN
+F 2 "Inductors_SMD:L_6.3x6.3_H3" H 5700 4950 50  0001 C CNN
+F 3 "~" H 5700 4950 50  0001 C CNN
+	1    5700 4950
 	0    -1   -1   0
 $EndComp
@@
 F 0 "R12" H 5334 5146 50  0000 L CNN
 F 1 "?" H 5325 5050 50  0000 L CNN
-F 2 "" H 5275 5100 50  0001 C CNN
+F 2 "Resistors_SMD:R_0805" H 5275 5100 50  0001 C CNN
 F 3 "~" H 5275 5100 50  0001 C CNN
 	1    5275 5100
@@
 Connection ~ 5475 4950
 Wire Wire Line
-	5475 4950 5675 4950
+	5475 4950 5600 4950
 Wire Wire Line
 	5875 5400 5925 5400
@@
 	5925 5400 5925 4950
 Wire Wire Line
-	5925 4950 5875 4950
+	5925 4950 5800 4950
 Wire Wire Line
 	6000 4950 5925 4950
@@
 F 0 "R14" H 6434 5846 50  0000 L CNN
 F 1 "1k5" H 6425 5750 50  0000 L CNN
-F 2 "" H 6375 5800 50  0001 C CNN
+F 2 "Resistors_SMD:R_0805" H 6375 5800 50  0001 C CNN
 F 3 "~" H 6375 5800 50  0001 C CNN
 	1    6375 5800
@@
 F 0 "R13" H 6434 5421 50  0000 L CNN
 F 1 "2k4" H 6425 5325 50  0000 L CNN
-F 2 "" H 6375 5375 50  0001 C CNN
+F 2 "Resistors_SMD:R_0805" H 6375 5375 50  0001 C CNN
 F 3 "~" H 6375 5375 50  0001 C CNN
 	1    6375 5375
@@
 F 0 "C8" H 4841 2246 50  0000 L CNN
 F 1 "10uF" H 4841 2155 50  0000 L CNN
-F 2 "" H 4750 2200 50  0001 C CNN
+F 2 "Capacitors_SMD:C_1210" H 4750 2200 50  0001 C CNN
 F 3 "~" H 4750 2200 50  0001 C CNN
 	1    4750 2200
@@
 F 0 "C12" H 6716 5646 50  0000 L CNN
 F 1 "10uF" H 6716 5555 50  0000 L CNN
-F 2 "" H 6625 5600 50  0001 C CNN
+F 2 "Capacitors_SMD:C_1210" H 6625 5600 50  0001 C CNN
 F 3 "~" H 6625 5600 50  0001 C CNN
 	1    6625 5600
@@
 F 0 "D1" V 4925 2900 50  0000 R CNN
 F 1 "LED" V 4825 2950 50  0000 R CNN
-F 2 "LEDs:LED_0603" H 4850 2725 50  0001 C CNN
+F 2 "LEDs:LED_0805" H 4850 2725 50  0001 C CNN
 F 3 "~" H 4850 2725 50  0001 C CNN
 	1    4850 2725
@@
 F 0 "D2" V 5089 2608 50  0000 R CNN
 F 1 "LED" V 4998 2608 50  0000 R CNN
-F 2 "LEDs:LED_0603" H 5050 2725 50  0001 C CNN
+F 2 "LEDs:LED_0805" H 5050 2725 50  0001 C CNN
 F 3 "~" H 5050 2725 50  0001 C CNN
 	1    5050 2725
@@
 	5050 2575 5050 2525
 Connection ~ 5050 2525
+$Comp
+L device:CP1_Small C?
+U 1 1 5CC8A14B
+P 6825 3550
+AR Path="/5CC8A14B" Ref="C?"  Part="1"
+AR Path="/5C948828/5CC8A14B" Ref="C11"  Part="1"
+F 0 "C11" H 6916 3596 50  0000 L CNN
+F 1 "10uF" H 6916 3505 50  0000 L CNN
+F 2 "Capacitors_SMD:C_1210" H 6825 3550 50  0001 C CNN
+F 3 "~" H 6825 3550 50  0001 C CNN
+	1    6825 3550
+	1    0    0    -1
+$EndComp
+Text Notes 4925 1600 0    50   ~ 0
+footprint ok
+$Comp
+L MLAB_HEADER:HEADER_1x02 J6
+U 1 1 5CCC104E
+P 7675 3650
+F 0 "J6" H 7753 3708 60  0000 L CNN
+F 1 "HEADER_1x02" H 7753 3602 60  0000 L CNN
+F 2 "Mlab_Pin_Headers:Straight_1x02" H 7753 3549 60  0001 L CNN
+F 3 "" H 7675 3700 60  0000 C CNN
+	1    7675 3650
+	1    0    0    -1
+$EndComp
+Wire Wire Line
+	7475 3600 7325 3600
+Wire Wire Line
+	7325 3600 7325 3250
+Connection ~ 7325 3250
+Wire Wire Line
+	7325 3250 6825 3250
+Wire Wire Line
+	7475 3700 7325 3700
+Wire Wire Line
+	7325 3700 7325 4050
+Connection ~ 7325 4050
+Wire Wire Line
+	7325 4050 7475 4050
 $EndSCHEMATC
