File: HW/SAR-APRS/Power.sch (KiCad schematic (older format))
At the start: 24 parts, among them J6 HEADER_1x02, Q2 2N7002, Q3 2N7002, U2 TP4056, U3 DW01x, U4 TPS61023

Commit message: ibom added
Parts:
- R13: value ? -> 500k
- R14: value ? -> 110k
Changed lines of the file:
@@
 AR Path="/5C948828/5C95AD18" Ref="R14"  Part="1"
 F 0 "R14" H 5209 6196 50  0000 L CNN
-F 1 "?" H 5200 6100 50  0000 L CNN
+F 1 "110k" H 5200 6100 50  0000 L CNN
 F 2 "Resistors_SMD:R_0805" H 5150 6150 50  0001 C CNN
 F 3 "~" H 5150 6150 50  0001 C CNN
@@
 AR Path="/5C948828/5C95AD1E" Ref="R13"  Part="1"
 F 0 "R13" H 5209 5896 50  0000 L CNN
-F 1 "?" H 5200 5800 50  0000 L CNN
+F 1 "500k" H 5200 5800 50  0000 L CNN
 F 2 "Resistors_SMD:R_0805" H 5150 5850 50  0001 C CNN
 F 3 "~" H 5150 5850 50  0001 C CNN
